File: hardware/BODAQS shield v1/BODAQS shield v1.kicad_sch (KiCad schematic)
At the start: 60 parts, among them J1 Analog Input 1, J10 Reset, J2 Reset, J3 Bar switch, J4 Navigation pad, J5 I2C Breakout, J6 Analog Input 2, J7 Analog Input 3, J8 Analog Input 4, J9 UART Breakout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

Commit message: Support SDMMA and SDFat
Parts:
- removed C14, C16: 10uF, Capacitor_THT:C_Disc_D9.0mm_W2.5mm_P5.00mm, symbol Device:C
- added TP1, TP2, TP3, TP4: TestPoint, Connector_Pin:Pin_D0.7mm_L6.5mm_W1.8mm_FlatFork, symbol Connector:TestPoint
- J10: value Reset -> Charge
Connections:
- net +3V3: now also TP1.1; no longer U1.27 (3V3EN)
- net A3V3: now also TP3.1
- net AGND: now also TP4.1
- net ANALOG1: now also U1.7 (GPIO15); no longer U1.10 (GPIO18)
- net ANALOG3: now also U1.10 (GPIO18); no longer U1.7 (GPIO15)
- net BUZZER: now also U1.16 (GPIO42); no longer U1.12 (GPIO11)
- net GND: now also TP2.1
