File: hardware/BODAQS shield v2 SMD/BODAQS shield v2 SMD.kicad_sch (KiCad schematic)
At the start: 61 parts, among them J1 Analog Input 1, J10 Charge, J2 Reset, J3 Bar switch, J4 Navigation pad, J5 I2C Breakout, J6 Analog Input 2, J7 Analog Input 3, J8 Analog Input 4, J9 UART Breakout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

Commit message: File cleanup
Parts:
- removed C17: 10uF, Capacitor_SMD:C_0603_1608Metric_Pad1.08x0.95mm_HandSolder, symbol Device:C
- removed C19, C21: 100nF, Capacitor_SMD:C_0603_1608Metric_Pad1.08x0.95mm_HandSolder, symbol Device:C
- removed FB1: FerriteBead, Inductor_THT:L_Axial_L11.0mm_D4.5mm_P15.24mm_Horizontal_Fastron_MECC, symbol Device:FerriteBead
Connections:
- net +3V3: no longer C20.1, NT1.1
- net BATTERY: now reaches U1.28 (VBAT)
- net BATTERY: now also C20.1, NT1.1
- no-connect marks 8 -> 7
Other:
- moved on the sheet: C18, TP3
