File: hardware/BODAQS shield Proto E/BODAQS shield Proto E.kicad_sch (KiCad schematic)
At the start: 52 parts, among them J1 Analog Input 1, J3 Bar switch, J4 Navigation pad, J5 I2C Breakout, J6 Analog Input 2, J7 Analog Input 3, J8 Analog Input 4, J9 UART Breakout, U2 MCP6004, U4 LD1117V33

Commit message: Finish hardware prototype E design (TH and SMD)
Parts:
- C1, C10, C4, C7: value 220nF -> 47nF
- C12, C3, C6, C9: value 100nF -> 10nF
- R13, R14, R18, R19, R3, R4, R8, R9: value 2K -> 4.7K
Changed lines of the file:
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@@
 			)
 		)
-		(property "Value" "2K"
+		(property "Value" "4.7K"
 			(at 162.56 39.37 90)
 			(effects
@@
 			)
 		)
-		(property "Value" "2K"
+		(property "Value" "4.7K"
 			(at 255.27 39.37 90)
 			(effects
@@
 			)
 		)
-		(property "Value" "2K"
+		(property "Value" "4.7K"
 			(at 162.56 96.52 90)
 			(effects
@@
 			)
 		)
-		(property "Value" "220nF"
+		(property "Value" "47nF"
 			(at 242.57 111.7599 0)
 			(effects
@@
 			)
 		)
-		(property "Value" "100nF"
+		(property "Value" "10nF"
 			(at 210.82 111.7599 0)
 			(effects
@@
 			)
 		)
-		(property "Value" "100nF"
+		(property "Value" "10nF"
 			(at 118.11 111.7599 0)
 			(effects
@@
 			)
 		)
-		(property "Value" "220nF"
+		(property "Value" "47nF"
 			(at 242.57 54.6099 0)
 			(effects
@@
 			)
 		)
-		(property "Value" "100nF"
+		(property "Value" "10nF"
 			(at 118.11 54.6099 0)
 			(effects
@@
 			)
 		)
-		(property "Value" "220nF"
+		(property "Value" "47nF"
 			(at 149.86 111.7599 0)
 			(effects
@@
 			)
 		)
-		(property "Value" "220nF"
+		(property "Value" "47nF"
 			(at 149.86 54.6099 0)
 			(effects
@@
 			)
 		)
-		(property "Value" "2K"
+		(property "Value" "4.7K"
 			(at 152.4 39.37 90)
 			(effects
@@
 			)
 		)
-		(property "Value" "2K"
+		(property "Value" "4.7K"
 			(at 245.11 39.37 90)
 			(effects
@@
 			)
 		)
-		(property "Value" "2K"
+		(property "Value" "4.7K"
 			(at 245.11 96.52 90)
 			(effects
@@
 			)
 		)
-		(property "Value" "2K"
+		(property "Value" "4.7K"
 			(at 152.4 96.52 90)
 			(effects
@@
 			)
 		)
-		(property "Value" "100nF"
+		(property "Value" "10nF"
 			(at 210.82 54.6099 0)
 			(effects
@@
 			)
 		)
-		(property "Value" "2K"
+		(property "Value" "4.7K"
 			(at 255.27 96.52 90)
 			(effects
