File: hardware/BODAQS shield Proto E SMD/BODAQS shield Proto E SMD.kicad_pcb (KiCad board)
At the start: 2 copper layers, 47.3 x 56.5 mm, 48 parts, among them J1 Analog1, J3 Bar switch, J4 Nav pad, J5 I2C, J6 Analog2, J7 Analog3, J8 Analog4, J9 UART, U2 MCP6004, U4 LD1117V33

Commit message: Finish hardware prototype E design (TH and SMD)
Parts:
- C1, C10, C4, C7: value 220nF -> 47nF
- C12, C3, C6, C9: value 100nF -> 10nF
- C17: footprint Capacitor_SMD:C_0603_1608Metric -> Capacitor_SMD:C_1206_3216Metric
- J3: value Bar switch -> Bar
- J4: value Nav pad -> Navigation
- J9: value UART -> UART Breakout
- R13, R14, R19, R3, R4, R8, R9: value 2K -> 4.7K
- R18: value 2K -> 4.7K'
- U4: value LD1117V33 -> LDL1117S33R
- moved C17 2.22 mm to (182.0, 98.3)
- moved C15 1.71 mm to (180.1, 100.2)
Routing:
- net GND: track 1.31 -> 14.5 mm, vias 1 -> 10
- net AGND: track 16.1 -> 7.00 mm, vias 6 -> 9
- net Net-(U2B-+): track 29.4 -> 31.2 mm
- net A3V3: track 65.0 -> 66.1 mm
- added copper zone on B.Cu, net AGND
