File: hardware/BODAQS shield Proto E SMD/BODAQS shield Proto E SMD.kicad_sch (KiCad schematic)
At the start: 48 parts, among them J1 Analog Input 1, J3 Bar switch, J4 Navigation pad, J5 I2C Breakout, J6 Analog Input 2, J7 Analog Input 3, J8 Analog Input 4, J9 UART Breakout, U2 MCP6004, U4 LD1117V33

Commit message: Finish hardware prototype E design (TH and SMD)
Parts:
- C1, C10, C4, C7: value 220nF -> 47nF
- C12, C3, C6, C9: value 100nF -> 10nF
- C17: footprint Capacitor_SMD:C_0603_1608Metric -> Capacitor_SMD:C_0805_2012Metric
- J1: value Analog Input 1 -> Analog1
- J3: value Bar switch -> Bar
- J4: value Navigation pad -> Navigation
- J5: value I2C Breakout -> I2C
- J6: value Analog Input 2 -> Analog2
- J7: value Analog Input 3 -> Analog3
- J8: value Analog Input 4 -> Analog4
- R13, R14, R19, R3, R4, R8, R9: value 2K -> 4.7K
- R18: value 2K -> 4.7K'
- U4: value LD1117V33 -> LDL1117S33R
Changed lines of the file:
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@@
 			)
 		)
-		(property "Value" "2K"
+		(property "Value" "4.7K"
 			(at 162.56 39.37 90)
 			(effects
@@
 			)
 		)
-		(property "Value" "Analog Input 4"
+		(property "Value" "Analog4"
 			(at 177.8 101.5999 0)
 			(effects
@@
 			)
 		)
-		(property "Value" "Bar switch"
+		(property "Value" "Bar"
 			(at 22.86 45.72 0)
 			(effects
@@
 			)
 		)
-		(property "Value" "2K"
+		(property "Value" "4.7K"
 			(at 255.27 39.37 90)
 			(effects
@@
 			)
 		)
-		(property "Value" "Analog Input 2"
+		(property "Value" "Analog2"
 			(at 270.51 101.5999 0)
 			(effects
@@
 			)
 		)
-		(property "Value" "2K"
+		(property "Value" "4.7K'"
 			(at 162.56 96.52 90)
 			(effects
@@
 			)
 		)
-		(property "Value" "I2C Breakout"
+		(property "Value" "I2C"
 			(at 22.86 24.13 0)
 			(effects
@@
 			)
 		)
-		(property "Value" "220nF"
+		(property "Value" "47nF"
 			(at 242.57 111.7599 0)
 			(effects
@@
 			)
 		)
-		(property "Value" "Navigation pad"
+		(property "Value" "Navigation"
 			(at 50.8 22.86 0)
 			(effects
@@
 			)
 		)
-		(property "Value" "100nF"
+		(property "Value" "10nF"
 			(at 210.82 111.7599 0)
 			(effects
@@
 			)
 		)
-		(property "Value" "100nF"
+		(property "Value" "10nF"
 			(at 118.11 111.7599 0)
 			(effects
@@
 			)
 		)
-		(property "Value" "220nF"
+		(property "Value" "47nF"
 			(at 242.57 54.6099 0)
 			(effects
@@
 			)
 		)
-		(property "Value" "100nF"
+		(property "Value" "10nF"
 			(at 118.11 54.6099 0)
 			(effects
@@
 			)
 		)
-		(property "Value" "220nF"
+		(property "Value" "47nF"
 			(at 149.86 111.7599 0)
 			(effects
@@
 			)
 		)
-		(property "Value" "220nF"
+		(property "Value" "47nF"
 			(at 149.86 54.6099 0)
 			(effects
@@
 			)
 		)
-		(property "Footprint" "Capacitor_SMD:C_0603_1608Metric"
+		(property "Footprint" "Capacitor_SMD:C_0805_2012Metric"
 			(at 72.0852 97.79 0)
 			(effects
@@
 			)
 		)
-		(property "Value" "2K"
+		(property "Value" "4.7K"
 			(at 152.4 39.37 90)
 			(effects
@@
 			)
 		)
-		(property "Value" "2K"
+		(property "Value" "4.7K"
 			(at 245.11 39.37 90)
 			(effects
@@
 			)
 		)
-		(property "Value" "2K"
+		(property "Value" "4.7K"
 			(at 245.11 96.52 90)
 			(effects
@@
 			)
 		)
-		(property "Value" "2K"
+		(property "Value" "4.7K"
 			(at 152.4 96.52 90)
 			(effects
@@
 			)
 		)
-		(property "Value" "100nF"
+		(property "Value" "10nF"
 			(at 210.82 54.6099 0)
 			(effects
@@
 			)
 		)
-		(property "Value" "2K"
+		(property "Value" "4.7K"
 			(at 255.27 96.52 90)
 			(effects
@@
 			)
 		)
-		(property "Value" "Analog Input 3"
+		(property "Value" "Analog3"
 			(at 177.8 44.4499 0)
 			(effects
@@
 			)
 		)
-		(property "Value" "Analog Input 1"
+		(property "Value" "Analog1"
 			(at 270.51 44.4499 0)
 			(effects
@@
 			)
 		)
-		(property "Value" "LD1117V33"
+		(property "Value" "LDL1117S33R"
 			(at 52.07 78.74 0)
 			(effects
@@
 			)
 		)
-		(property "Datasheet" "https://www.st.com/resource/en/datasheet/ld1117.pdf"
+		(property "Datasheet" ""
 			(at 54.61 88.9 0)
 			(effects
