File: hardware/BODAQS shield SMD Proto F/BODAQS shield SMD Proto F.kicad_sch (KiCad schematic)
At the start: 32 parts, among them J1 Analog1, J2 Analog2, J3 Analog3, J4 Analog4, J5 Bar, J6 I2C1, J7 UART, J8 Navigation, J9 SPI, U2 MCP6004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

Commit message: Update build guide
Parts:
- added U3: TPS7A2033PDBVR, TPS7A2033PDBVR:SOT95P280X145-5N, symbol TPS7A2033PDBVR:TPS7A2033PDBVR
- added U5: ADS1220IRVAR, ADS1220IRVAR:QFN50P350X350X100-17N, symbol ADS1220IRVAR:ADS1220IRVAR
