File: hardware/BODAQS shield SMD Proto F/BODAQS shield SMD Proto F.kicad_sch (KiCad schematic)
At the start: 36 parts, among them J1 Analog1, J10 I2C0, J2 Analog2, J3 Analog3, J4 Analog4, J5 Bar, J6 I2C1, J7 UART, J8 Navigation, U2 MCP6004, U3 TPS7A2033PDBVR, U5 ADS1220IRVAR

Commit message: More work on hardware design
Parts:
- removed U3: TPS7A2033PDBVR, TPS7A2033PDBVR:SOT95P280X145-5N, symbol TPS7A2033PDBVR:TPS7A2033PDBVR
- removed U5: ADS1220IRVAR, ADS1220IRVAR:QFN50P350X350X100-17N, symbol ADS1220IRVAR:ADS1220IRVAR
- J1, J2, J3, J4, J5: footprint Connector_PinHeader_2.00mm:PinHeader_1x03_P2.00mm_Vertical -> Connector_JST:JST_PH_S3B-PH-SM4-TB_1x03-1MP_P2.00mm_Horizontal
- J6: renamed from J10; footprint Connector_PinHeader_2.00mm:PinHeader_1x04_P2.00mm_Vertical -> Connector_JST:JST_PH_S4B-PH-SM4-TB_1x04-1MP_P2.00mm_Horizontal
- J7: renamed from J6; footprint Connector_PinHeader_2.00mm:PinHeader_1x04_P2.00mm_Vertical -> Connector_JST:JST_PH_S4B-PH-SM4-TB_1x04-1MP_P2.00mm_Horizontal
- J8: renamed from J7; footprint Connector_PinHeader_2.54mm:PinHeader_1x04_P2.54mm_Vertical -> Connector_JST:JST_PH_S4B-PH-SM4-TB_1x04-1MP_P2.00mm_Horizontal
- U1: footprint Module:Adafruit_Feather -> Module:Adafruit_Feather_32u4_RFM
- renumbered C2 to C1, C3 to C2, C5 to C3, C7 to C4, C21 to C6, C17 to C7, C9 to C8, J8 to J9, R8 to R10, R7 to R11, R9 to R3, R3 to R5, R10 to R6, R6 to R7, R5 to R8, R11 to R9
