File: hardware/BODAQS shield SMD Proto F/BODAQS shield SMD Proto F.kicad_pcb (KiCad board)
At the start: 4 copper layers, 47.3 x 56.5 mm, 32 parts, among them J1 Analog1, J2 Analog2, J3 Analog3, J4 Analog4, J5 Bar, J6 I2C1, J7 UART, J8 Navigation, J9 SPI, U2 MCP6004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

Commit message: Progress in rev F of PCB
Parts:
- removed C1, C4, C6, C8: 100nF, Capacitor_SMD:C_0603_1608Metric
- removed J9: SPI, Connector_PinHeader_2.54mm:PinHeader_1x06_P2.54mm_Vertical
- removed U4: LDL1117S33R, Package_TO_SOT_SMD:SOT-223-3_TabPin2
- added D1: BAT60A, Diode_SMD:D_SOD-323, F.Cu at (162.1, 121.9)
- added D2: BAT60A, Diode_SMD:D_SOD-323, F.Cu at (162.1, 124.0)
- added J10: I2C0, Connector_PinHeader_2.00mm:PinHeader_1x04_P2.00mm_Vertical, F.Cu at (153.1, 87.4)
- added R10: 10K, Resistor_SMD:R_0603_1608Metric, F.Cu at (173.8, 97.6)
- added R11: 10K, Resistor_SMD:R_0603_1608Metric, F.Cu at (173.8, 99.9)
- added R12: 10K, Resistor_SMD:R_0603_1608Metric, F.Cu at (173.8, 104.7)
- added R9: 10K, Resistor_SMD:R_0603_1608Metric, F.Cu at (173.8, 109.9)
- added U3: TPS7A2033PDBVR, Package_TO_SOT_SMD:SOT-23-5, F.Cu at (179.8, 118.0)
- C17: value 10uF -> 2.2uF
- C21: value 100nF -> 2.2uF
- R1, R4, R6, R8: value 1.6K -> 10K
- moved J6 33.2 mm to (154.1, 126.0), turned to -90 degrees
- moved J5 8.68 mm to (146.9, 73.8), turned to -90 degrees
Connections:
- C21 pad 1: VBAT -> VIN
- NT1 pad 1: VBAT -> VIN
- U1 pad 11: SCK -> unconnected-(U1-12/SCK-Pad11)
- U1 pad 12: PICO -> unconnected-(U1-11/PICO-Pad12)
- U1 pad 13: POCI -> unconnected-(U1-13/POCI-Pad13)
- U1 pad 16: CS -> EN
- U1 pad 17: unconnected-(U1-SDA/8-Pad17) -> SDA0
- U1 pad 18: unconnected-(U1-SCL/9-Pad18) -> SCL0
- U1 pad 26: unconnected-(U1-VUSB-Pad26) -> VUSB
Routing:
- net unconnected-(U1-13/POCI-Pad13): track 0.00 -> 8.54 mm
- net unconnected-(U1-12/SCK-Pad11): track 0.00 -> 8.54 mm
- net SCK: track 8.54 -> 0.00 mm
- net POCI: track 8.54 -> 0.00 mm
- net unconnected-(U1-11/PICO-Pad12): track 0.00 -> 8.54 mm
- net PICO: track 8.54 -> 0.00 mm
- net VBAT: track 9.62 -> 2.32 mm, vias 2 -> 1
- net A3V3: track 21.8 -> 14.5 mm
- net VIN: track 0.00 -> 6.65 mm
- net EN: track 0.00 -> 5.01 mm
- net CS: track 5.01 -> 0.00 mm
- net GND: track 38.8 -> 37.2 mm
- removed copper zone on In2.Cu, net VBAT
Other:
- board text removed: "Sparkfun ESP32 Thing Plus S3"

Commit message: Merge branch 'mobile-fixup' of https://github.com/benconnor1972/BODAQS
Parts:
- moved J7 19.3 mm to (161.2, 107.2), turned to -90 degrees
Changed lines of the file:
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@@
 	(footprint "Connector_PinHeader_2.54mm:PinHeader_1x04_P2.54mm_Vertical"
 		(layer "F.Cu")
-		(at 141.9 107.5 180)
+		(at 161.24 107.2 -90)
 		(descr "Through hole straight pin header, 1x04, 2.54mm pitch, single row")
 		(tags "Through hole pin header THT 1x04 2.54mm single row")
 		(property "Reference" "J7"
-			(at 0 -2.38 0)
+			(at 0 -2.38 90)
 			(layer "F.SilkS")
 			(hide yes)
@@
 		)
 		(property "Value" "UART"
-			(at 2.6 0.11 90)
+			(at 2.6 0.11 0)
 			(layer "F.Fab")
 			(effects
@@
 		)
 		(property "Datasheet" "~"
-			(at 0 0 0)
+			(at 0 0 90)
 			(layer "F.Fab")
 			(hide yes)
@@
 		)
 		(property "Description" "Generic connector, single row, 01x04, script generated (kicad-library-utils/schlib/autogen/connector/)"
-			(at 0 0 0)
+			(at 0 0 90)
 			(layer "F.Fab")
 			(hide yes)
@@
 		(attr through_hole)
 		(fp_line
+			(start -1.38 9)
+			(end 1.38 9)
+			(stroke
+				(width 0.12)
+				(type solid)
+			)
+			(layer "F.SilkS")
+		)
+		(fp_line
+			(start -1.38 1.27)
+			(end -1.38 9)
+			(stroke
+				(width 0.12)
+				(type solid)
+			)
+			(layer "F.SilkS")
+		)
+		(fp_line
+			(start -1.38 1.27)
+			(end 1.38 1.27)
+			(stroke
+				(width 0.12)
+				(type solid)
+			)
+			(layer "F.SilkS")
+		)
+		(fp_line
 			(start 1.38 1.27)
 			(end 1.38 9)
@@
 		)
 		(fp_line
-			(start -1.38 9)
-			(end 1.38 9)
-			(stroke
-				(width 0.12)
-				(type solid)
-			)
-			(layer "F.SilkS")
-		)
-		(fp_line
-			(start -1.38 1.27)
-			(end 1.38 1.27)
-			(stroke
-				(width 0.12)
-				(type solid)
-			)
-			(layer "F.SilkS")
-		)
-		(fp_line
-			(start -1.38 1.27)
-			(end -1.38 9)
-			(stroke
-				(width 0.12)
-				(type solid)
-			)
-			(layer "F.SilkS")
-		)
-		(fp_line
 			(start -1.38 0)
 			(end -1.38 -1.38)
@@
 		)
 		(fp_line
+			(start -1.77 9.39)
+			(end 1.77 9.39)
+			(stroke
+				(width 0.05)
+				(type solid)
+			)
+			(layer "F.CrtYd")
+		)
+		(fp_line
 			(start 1.77 9.39)
 			(end 1.77 -1.77)
@@
 		)
 		(fp_line
+			(start -1.77 -1.77)
+			(end -1.77 9.39)
+			(stroke
+				(width 0.05)
+				(type solid)
+			)
+			(layer "F.CrtYd")
+		)
+		(fp_line
 			(start 1.77 -1.77)
 			(end -1.77 -1.77)
@@
 		)
 		(fp_line
-			(start -1.77 9.39)
-			(end 1.77 9.39)
-			(stroke
-				(width 0.05)
-				(type solid)
-			)
-			(layer "F.CrtYd")
-		)
-		(fp_line
-			(start -1.77 -1.77)
-			(end -1.77 9.39)
-			(stroke
-				(width 0.05)
-				(type solid)
-			)
-			(layer "F.CrtYd")
+			(start -1.27 8.89)
+			(end -1.27 -0.635)
+			(stroke
+				(width 0.1)
+				(type solid)
+			)
+			(layer "F.Fab")
 		)
 		(fp_line
@@
 		)
 		(fp_line
+			(start -1.27 -0.635)
+			(end -0.635 -1.27)
+			(stroke
+				(width 0.1)
+				(type solid)
+			)
+			(layer "F.Fab")
+		)
+		(fp_line
+			(start -0.635 -1.27)
+			(end 1.27 -1.27)
+			(stroke
+				(width 0.1)
+				(type solid)
+			)
+			(layer "F.Fab")
+		)
+		(fp_line
 			(start 1.27 -1.27)
 			(end 1.27 8.89)
@@
 			(layer "F.Fab")
 		)
-		(fp_line
-			(start -0.635 -1.27)
-			(end 1.27 -1.27)
-			(stroke
-				(width 0.1)
-				(type solid)
-			)
-			(layer "F.Fab")
-		)
-		(fp_line
-			(start -1.27 8.89)
-			(end -1.27 -0.635)
-			(stroke
-				(width 0.1)
-				(type solid)
-			)
-			(layer "F.Fab")
-		)
-		(fp_line
-			(start -1.27 -0.635)
-			(end -0.635 -1.27)
-			(stroke
-				(width 0.1)
-				(type solid)
-			)
-			(layer "F.Fab")
-		)
 		(fp_text user "${REFERENCE}"
-			(at 0 3.81 90)
+			(at 0 3.81 0)
 			(layer "F.Fab")
 			(effects
@@
 		)
 		(pad "1" thru_hole rect
-			(at 0 0 180)
+			(at 0 0 270)
 			(size 1.7 1.7)
 			(drill 1)
@@
 		)
 		(pad "2" thru_hole circle
-			(at 0 2.54 180)
+			(at 0 2.54 270)
 			(size 1.7 1.7)
 			(drill 1)
@@
 		)
 		(pad "3" thru_hole circle
-			(at 0 5.08 180)
+			(at 0 5.08 270)
 			(size 1.7 1.7)
 			(drill 1)
@@
 		)
 		(pad "4" thru_hole circle
-			(at 0 7.62 180)
-			(size 1.7 1.7)
-			(drill 1)
+			(at 0 7.62 270)
+			(size 1.7 1.7)
+			(drill 1)
